File: client/jakesensors_client/nRF24L01-Chip-v13.sch (EAGLE design)
At the start: 25 parts, among them IC1 BME280, Q1 16MHz, U1 NRF24, U2 ATMEGA328P-MU, U3 APDS-9960, U4 RPI-103X, Y1 ANTENNA2SMD5

Commit message: commit
Parts:
- added R3: 39, SparkFun:RESISTOR0402-RES
Connections:
- new net N$32: R3.1, U4.CATHODE
- net GND: now also R3.2; no longer U4.CATHODE
Changed lines of the file:
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@@
 <part name="P+7" library="SparkFun" deviceset="VCC" device=""/>
 <part name="GND16" library="SparkFun" deviceset="GND" device=""/>
+<part name="R3" library="SparkFun" deviceset="RESISTOR" device="0402-RES" value="39"/>
 </parts>
 <sheets>
@@
 <instance part="U4" gate="G$1" x="114.3" y="162.56"/>
 <instance part="P+7" gate="1" x="88.9" y="165.1"/>
-<instance part="GND16" gate="1" x="139.7" y="165.1"/>
+<instance part="GND16" gate="1" x="157.48" y="165.1"/>
+<instance part="R3" gate="G$1" x="142.24" y="167.64"/>
 </instances>
 <busses>
@@
 </segment>
 <segment>
-<pinref part="U4" gate="G$1" pin="CATHODE"/>
+<pinref part="R3" gate="G$1" pin="2"/>
 <pinref part="GND16" gate="1" pin="GND"/>
-<wire x1="132.08" y1="167.64" x2="139.7" y2="167.64" width="0.1524" layer="91"/>
+<wire x1="147.32" y1="167.64" x2="157.48" y2="167.64" width="0.1524" layer="91"/>
 </segment>
 </net>
@@
 </segment>
 </net>
+<net name="N$32" class="0">
+<segment>
+<pinref part="U4" gate="G$1" pin="CATHODE"/>
+<pinref part="R3" gate="G$1" pin="1"/>
+<wire x1="132.08" y1="167.64" x2="137.16" y2="167.64" width="0.1524" layer="91"/>
+</segment>
+</net>
