File: server/eagle_proj/nRF24L01-Chip-v13.brd (EAGLE design)
At the start: 66.8 x 80.5 mm, 14 parts, among them IC1 7805DT

Commit message: Server updates
Parts:
- added R1, R2: 10k, resistor:R0402
Connections:
- new net N$21: JP2.8, R1.1, U2.14
- net GND: now also JP2.11, JP2.9
- net N$11: now also JP2.5
- net N$12: now also JP2.6
- net N$13: now also JP2.3
- net N$14: now also R2.2
- net N$15: now also U2.7; no longer U2.8
- net N$16: now also U2.2; no longer U2.7
- net N$17: now also U2.1; no longer U2.2
- net N$18: now also U2.32; no longer U2.1
- net N$19: now also U2.31; no longer U2.32
- net N$20: now also U2.30; no longer U2.31
- net N$3: now also U2.13; no longer U2.14
- net N$4: now also U2.12; no longer U2.13
- net N$5: now also U2.11; no longer U2.12
- net N$6: now also U2.10; no longer U2.11
- net N$7: now also U2.9; no longer U2.10
- net N$9: now also U2.8; no longer U2.9
- net VCC: now also JP2.10, R1.2, R2.1
Routing:
- net GND: track 86.8 -> 276.0 mm, vias 0 -> 3
- net VCC: track 51.4 -> 144.6 mm, vias 3 -> 4
- net N$21: track 0.00 -> 79.9 mm
- net N$11: track 28.4 -> 56.9 mm, vias 2 -> 3
- net N$13: track 27.9 -> 56.4 mm
- net N$12: track 40.2 -> 62.1 mm, vias 0 -> 1
- net N$19: track 48.2 -> 51.3 mm
- net N$18: track 52.5 -> 55.5 mm
- net N$16: track 42.5 -> 45.0 mm
- net N$20: track 43.4 -> 45.9 mm
- net N$14: track 29.4 -> 31.5 mm
- net N$3: track 34.6 -> 34.1 mm
- net N$17: track 39.3 -> 39.8 mm
- net N$15: track 48.5 -> 49.0 mm
- net N$4: track 29.5 -> 29.0 mm
- added copper zone on layer 1, net N$8
