File: server/eagle_proj/nRF24L01-Chip-v13.sch (EAGLE design)
At the start: 12 parts, among them IC1 BME280, U2 ATMEGA328P-MU, U3 APDS-9960, U4 RPI-103X

Commit message: start of server
Parts:
- removed R3: 39, SparkFun:RESISTOR0402-RES
- removed U$1: NRF24L01+, NRF:NRF24L01+
- removed U3: APDS-9960, SparkFun-Sensors:APDS-9960
- removed U4: RPI-103X, SparkFun-Sensors:RPI-103X
- removed V1: (no value), battery_xtra:TAKACHI_BATT-CR123A
- added JP2: (no value), pinhead:PINHD-2X6/90
- added LED2, LED3, LED4, LED5, LED6: (no value), LilyPad-Wearables:LED1206
- added U$2: NRF24L01+, nrf24L01:NRF24L01+
- IC1: value BME280 -> 7805DT; device bosch-bme280:BME280 -> linear:7805DT
- JP1: device pinhead+:PINHD-1X31X03_SMT -> pinhead+:PINHD-2X12SMT
- LED1: value LED-0402 -> (none); device pel_dipol_comp:LED-0402 -> LilyPad-Wearables:LED1206
Connections:
- removed net N$21: U$1.5.SCK, U2.PD7
- removed net N$23: IC1.CSB
- removed net N$24: JP1.3
- removed net N$25: JP1.1
- removed net N$28: S1.1
- removed net N$29: U4.ANODE
- removed net N$30: U4.E1
- removed net N$31: U2.PB7, U4.E2
- removed net N$32: R3.1, U4.CATHODE
- removed net N$37: U$1.7.MISO, U2.PB1
- removed net N$8: IC1.SDO
- new net N$20: S1.1, U2.PD1
- new net N$3: U$2.CE, U2.PB2
- new net N$4: U$2.SCK, U2.PB1
- new net N$5: U$2.IRQ, U$2.MISO, U2.PB0
- new net N$6: U$2.MOSI, U2.PD7
- new net N$7: U$2.CSN, U2.PD6
- new net N$9: LED5.A, U2.PD5
- net GND: now also JP1.1, JP1.23, JP1.24, LED2.C, LED3.C, LED4.C, LED5.C, LED6.C, U$2.GND; no longer R3.2, U3.GND, V1.-
- net N$1: now also IC1.VI, JP1.17, JP1.18, JP1.7, JP1.8; no longer U$1.6.MOSI, U2.PB0
- net N$15: now also LED6.A, U2.PB7; no longer U2.PC4, U3.SDA
- net N$16: now also LED4.A, U2.PB6; no longer U2.PC5, U3.SCL
- net N$17: now also LED3.A, U2.PD4; no longer IC1.SCK
- net N$18: now also LED2.A, U2.PD3; no longer U$1.3.CE, U2.PD5
- net N$19: now also LED1.A, U2.PD2; no longer U$1.4.CSN, U2.PD6
- net VCC: now also IC1.VO; no longer IC1.VDD, IC1.VDDIO, U3.INT, U3.VDD, U4.C1, U4.C2, V1.+
Other:
- moved on the sheet: LED1, P1, S1

Commit message: Server updates
Parts:
- added R1, R2: 10k, resistor:R-EU_R0402
Connections:
- new net N$21: JP2.8, R1.1, U2.PB2
- net GND: now also JP2.11, JP2.9
- net N$11: now also JP2.5
- net N$12: now also JP2.6
- net N$13: now also JP2.3
- net N$14: now also R2.2
- net N$15: now also U2.PB6; no longer U2.PB7
- net N$16: now also U2.PD4; no longer U2.PB6
- net N$17: now also U2.PD3; no longer U2.PD4
- net N$18: now also U2.PD2; no longer U2.PD3
- net N$19: now also U2.PD1; no longer U2.PD2
- net N$20: now also U2.PD0; no longer U2.PD1
- net N$3: now also U2.PB1; no longer U2.PB2
- net N$4: now also U2.PB0; no longer U2.PB1
- net N$5: now also U2.PD7; no longer U2.PB0
- net N$6: now also U2.PD6; no longer U2.PD7
- net N$7: now also U2.PD5; no longer U2.PD6
- net N$9: now also U2.PB7; no longer U2.PD5
- net VCC: now also JP2.10, R1.2, R2.1
Other:
- moved on the sheet: JP2, LED1, LED2, LED3, LED4, LED5, LED6
