File: server/eagle_proj/jake_server.sch (EAGLE design)
At the start: 16 parts, among them IC1 7805DT, U2 ATMEGA328P-MU

Commit message: Fix voltage regulator
Parts:
- removed IC1: 7805DT, linear:7805DT
- added C1: 100uf, SparkFun-Capacitors:CAP1206
- added IC2: REG1117, burr-brown:REG1117
Connections:
- net GND: now also C1.1, IC2.GND; no longer IC1.GND
- net N$1: now also C1.2, IC2.VIN; no longer IC1.VI
- net VCC: now also IC2.VOUT; no longer IC1.VO
Changed lines of the file:
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@@
 <part name="GND1" library="SparkFun" deviceset="GND" device=""/>
 <part name="JP1" library="pinhead+" deviceset="PINHD-2X12" device="SMT"/>
-<part name="IC1" library="linear" deviceset="78*" device="DT" technology="05"/>
 <part name="JP2" library="pinhead" deviceset="PINHD-2X6" device="/90"/>
 <part name="LED6" library="LilyPad-Wearables" deviceset="LED" device="1206"/>
@@
 <part name="R2" library="resistor" deviceset="R-EU_" device="R0402" value="10k"/>
 <part name="P+6" library="SparkFun" deviceset="VCC" device=""/>
+<part name="C1" library="SparkFun-Capacitors" deviceset="CAP" device="1206" value="100uf"/>
+<part name="IC2" library="burr-brown" deviceset="REG1117" device=""/>
 </parts>
 <sheets>
@@
 <instance part="GND1" gate="1" x="-10.16" y="-15.24"/>
 <instance part="JP1" gate="A" x="5.08" y="30.48"/>
-<instance part="IC1" gate="A1" x="15.24" y="0"/>
 <instance part="JP2" gate="A" x="167.64" y="88.9"/>
 <instance part="LED6" gate="G$1" x="76.2" y="86.36" rot="R90"/>
@@
 <instance part="R2" gate="G$1" x="93.98" y="43.18" rot="R90"/>
 <instance part="P+6" gate="1" x="81.28" y="35.56"/>
+<instance part="C1" gate="G$1" x="7.62" y="55.88" rot="R90"/>
+<instance part="IC2" gate="G$1" x="30.48" y="-12.7"/>
 </instances>
 <busses>
@@
 <junction x="-10.16" y="15.24"/>
 <pinref part="JP1" gate="A" pin="1"/>
-<wire x1="2.54" y1="43.18" x2="-10.16" y2="43.18" width="0.1524" layer="91"/>
+<wire x1="2.54" y1="43.18" x2="-7.62" y2="43.18" width="0.1524" layer="91"/>
 <pinref part="JP1" gate="A" pin="24"/>
+<wire x1="-7.62" y1="43.18" x2="-10.16" y2="43.18" width="0.1524" layer="91"/>
 <wire x1="10.16" y1="15.24" x2="2.54" y2="15.24" width="0.1524" layer="91"/>
 <junction x="2.54" y="15.24"/>
@@
 <wire x1="10.16" y1="43.18" x2="2.54" y2="43.18" width="0.1524" layer="91"/>
 <junction x="2.54" y="43.18"/>
-<pinref part="IC1" gate="A1" pin="GND"/>
 <wire x1="15.24" y1="-7.62" x2="-10.16" y2="-7.62" width="0.1524" layer="91"/>
 <junction x="-10.16" y="-7.62"/>
+<pinref part="C1" gate="G$1" pin="1"/>
+<wire x1="2.54" y1="55.88" x2="-7.62" y2="55.88" width="0.1524" layer="91"/>
+<wire x1="-7.62" y1="55.88" x2="-7.62" y2="43.18" width="0.1524" layer="91"/>
+<junction x="-7.62" y="43.18"/>
+<pinref part="IC2" gate="G$1" pin="GND"/>
+<wire x1="30.48" y1="-25.4" x2="15.24" y2="-25.4" width="0.1524" layer="91"/>
+<wire x1="15.24" y1="-25.4" x2="15.24" y2="-7.62" width="0.1524" layer="91"/>
 </segment>
 <segment>
@@
 <segment>
 <pinref part="GND3" gate="1" pin="GND"/>
-<wire x1="86.36" y1="124.46" x2="86.36" y2="120.65" width="0.1524" layer="91"/>
+<wire x1="86.36" y1="124.46" x2="86.36" y2="119.38" width="0.1524" layer="91"/>
 <pinref part="LED5" gate="G$1" pin="C"/>
 <pinref part="LED3" gate="G$1" pin="C"/>
 <pinref part="LED2" gate="G$1" pin="C"/>
-<wire x1="81.28" y1="119.38" x2="86.36" y2="116.84" width="0.1524" layer="91"/>
+<wire x1="81.28" y1="119.38" x2="86.36" y2="119.38" width="0.1524" layer="91"/>
 <pinref part="LED1" gate="G$1" pin="C"/>
 <wire x1="81.28" y1="121.92" x2="81.28" y2="119.38" width="0.1524" layer="91"/>
@@
 <wire x1="81.28" y1="114.3" x2="81.28" y2="116.84" width="0.1524" layer="91"/>
 <pinref part="U$2" gate="G$1" pin="GND"/>
-<wire x1="93.98" y1="120.65" x2="86.36" y2="120.65" width="0.1524" layer="91"/>
-<wire x1="86.36" y1="120.65" x2="86.36" y2="116.84" width="0.1524" layer="91"/>
+<wire x1="93.98" y1="120.65" x2="86.36" y2="119.38" width="0.1524" layer="91"/>
 <pinref part="LED4" gate="G$1" pin="C"/>
 <wire x1="81.28" y1="114.3" x2="81.28" y2="111.76" width="0.1524" layer="91"/>
 <junction x="81.28" y="114.3"/>
+<junction x="86.36" y="119.38"/>
 </segment>
 <segment>
@@
 </segment>
 <segment>
-<pinref part="IC1" gate="A1" pin="VO"/>
 <pinref part="P+3" gate="1" pin="VCC"/>
 <wire x1="25.4" y1="0" x2="33.02" y2="0" width="0.1524" layer="91"/>
+<junction x="33.02" y="0"/>
+<pinref part="IC2" gate="G$1" pin="VOUT"/>
+<wire x1="43.18" y1="-12.7" x2="43.18" y2="0" width="0.1524" layer="91"/>
+<wire x1="43.18" y1="0" x2="33.02" y2="0" width="0.1524" layer="91"/>
 </segment>
 <segment>
@@
 <wire x1="2.54" y1="22.86" x2="10.16" y2="22.86" width="0.1524" layer="91"/>
 <junction x="10.16" y="22.86"/>
-<pinref part="IC1" gate="A1" pin="VI"/>
-<wire x1="5.08" y1="0" x2="5.08" y2="10.16" width="0.1524" layer="91"/>
 <wire x1="5.08" y1="10.16" x2="17.78" y2="10.16" width="0.1524" layer="91"/>
 <wire x1="17.78" y1="10.16" x2="17.78" y2="22.86" width="0.1524" layer="91"/>
 <junction x="17.78" y="22.86"/>
-</segment>
-</net>
+<pinref part="C1" gate="G$1" pin="2"/>
+<wire x1="10.16" y1="55.88" x2="17.78" y2="55.88" width="0.1524" layer="91"/>
+<wire x1="17.78" y1="55.88" x2="17.78" y2="35.56" width="0.1524" layer="91"/>
+<junction x="17.78" y="35.56"/>
+<pinref part="IC2" gate="G$1" pin="VIN"/>
+<wire x1="17.78" y1="-12.7" x2="5.08" y2="-12.7" width="0.1524" layer="91"/>
+<wire x1="5.08" y1="-12.7" x2="5.08" y2="10.16" width="0.1524" layer="91"/>
+</segment>
+</net>
