File: client/eagle_proj/jake_client.brd (EAGLE design)
At the start: 20.5 x 44 mm, 12 parts, among them IC1 BME280, U4 RPI-103X

Commit message: Clared client todo
Parts:
- removed U$1: NRF24L01+, NRF:NRF24L01+
- added R1: 10k, SparkFun:0402-RES
- added U$2: NRF24L01+NRF24L01+MINI, nrf24L01:NRF24L01+MINI
Connections:
- net GND: now also U$2.GND
- net N$1: now also U$2.MOSI; no longer U$1.6
- net N$14: now also R1.1
- net N$18: now also U$2.CE; no longer U$1.3
- net N$19: now also U$2.CSN; no longer U$1.4
- net N$21: now also U$2.SCK; no longer U$1.5
- net N$37: now also U$2.MISO; no longer U$1.7
- net VCC: now also R1.2, U$2.VCC
Routing:
- net VCC: track 125.7 -> 135.8 mm
- net GND: track 129.6 -> 133.7 mm, vias 2 -> 3
- net N$14: track 18.6 -> 21.5 mm
Changed lines of the file:
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@@
 </element>
 <element name="R3" library="SparkFun" package="0402-RES" value="39" x="42.25" y="29.75" smashed="yes" rot="R180"/>
-<element name="U$1" library="NRF" package="NRF24L01+" value="NRF24L01+" x="44.4" y="36" rot="R90"/>
 <element name="V1" library="battery_xtra" package="TAKACHI_CR123A" value="" x="35.5" y="30"/>
+<element name="U$2" library="nrf24L01" package="NRF24L01+MINI" value="NRF24L01+NRF24L01+MINI" x="36.75" y="41.815" rot="R90"/>
+<element name="R1" library="SparkFun" package="0402-RES" value="10k" x="35.75" y="21" smashed="yes" rot="R270"/>
 </elements>
 <signals>
@@
 <wire x1="41.25" y1="12.5" x2="44.75" y2="12.5" width="1.016" layer="16"/>
 <wire x1="44.75" y1="12.5" x2="44.75" y2="29.75" width="1.016" layer="16"/>
-<wire x1="44.75" y1="29.75" x2="44.75" y2="47.75" width="1.016" layer="16"/>
+<wire x1="44.75" y1="29.75" x2="44.75" y2="39.25" width="1.016" layer="16"/>
+<wire x1="44.75" y1="39.25" x2="44.75" y2="47.75" width="1.016" layer="16"/>
 <wire x1="41.25" y1="8.93" x2="35.5" y2="8.93" width="1.016" layer="16"/>
 <wire x1="35.5" y1="8.93" x2="35.5" y2="9.68" width="1.016" layer="16"/>
@@
 <wire x1="27" y1="19.25" x2="27" y2="21.579" width="0.2" layer="1"/>
 <wire x1="27" y1="21.579" x2="27.46" y2="21.579" width="0.2" layer="1"/>
+<contactref element="U$2" pad="GND"/>
+<wire x1="44.6113" y1="38.9702" x2="42.75" y2="38.9702" width="0.2" layer="1"/>
+<wire x1="42.75" y1="38.9702" x2="42.75" y2="39.25" width="0.2" layer="1"/>
+<via x="42.75" y="39.25" extent="1-16" drill="0.3" shape="octagon"/>
+<wire x1="42.75" y1="39.25" x2="44.75" y2="39.25" width="0.2" layer="16"/>
 </signal>
 <signal name="VCC">
@@
 <wire x1="31.25" y1="17.75" x2="31.25" y2="17.025" width="0.2" layer="1"/>
 <wire x1="31.25" y1="17.025" x2="31.225" y2="17.025" width="0.2" layer="1"/>
+<contactref element="U$2" pad="VCC"/>
+<wire x1="44.6113" y1="37.7002" x2="41.5" y2="37.7002" width="0.2" layer="1"/>
+<wire x1="41.5" y1="37.7002" x2="41.5" y2="37.75" width="0.2" layer="1"/>
+<contactref element="R1" pad="2"/>
+<wire x1="35.75" y1="20.35" x2="35.75" y2="19.25" width="0.2" layer="1"/>
+<wire x1="35.75" y1="19.25" x2="33" y2="19.25" width="0.2" layer="1"/>
+<wire x1="33" y1="19.25" x2="33" y2="17" width="0.2" layer="1"/>
+<wire x1="33" y1="17" x2="32.25" y2="17" width="0.2" layer="1"/>
 </signal>
 <signal name="GND1">
@@
 <via x="36.5" y="23.75" extent="1-16" drill="0.3"/>
 <contactref element="U2" pad="29"/>
+<contactref element="R1" pad="1"/>
+<wire x1="35.75" y1="21.65" x2="35.75" y2="23.75" width="0.2" layer="1"/>
+<wire x1="35.75" y1="23.75" x2="36.5" y2="23.75" width="0.2" layer="1"/>
 <wire x1="35.75" y1="29.2862" x2="35.754" y2="29.2862" width="0" layer="19" extent="1-1"/>
 </signal>
@@
 <signal name="N$18">
 <contactref element="U2" pad="9"/>
-<contactref element="U$1" pad="3"/>
-<wire x1="44.4" y1="40.25" x2="43.25" y2="40.25" width="0.2" layer="1"/>
 <wire x1="43.25" y1="40.25" x2="43" y2="40.5" width="0.2" layer="1"/>
 <wire x1="43" y1="40.5" x2="43" y2="41.25" width="0.2" layer="1"/>
@@
 <wire x1="37.25" y1="39" x2="37.25" y2="34.502665625" width="0.2" layer="1"/>
 <wire x1="37.25" y1="34.502665625" x2="37.2526" y2="34.2138" width="0.2" layer="1"/>
+<contactref element="U$2" pad="CE"/>
+<wire x1="43.25" y1="40.25" x2="44.6113" y2="40.25" width="0.2" layer="1"/>
+<wire x1="44.6113" y1="40.25" x2="44.6113" y2="40.2402" width="0.2" layer="1"/>
 </signal>
 <signal name="N$19">
 <contactref element="U2" pad="10"/>
-<contactref element="U$1" pad="4"/>
-<wire x1="44.4" y1="41.5" x2="43.25" y2="41.5" width="0.2" layer="1"/>
 <wire x1="43.25" y1="41.5" x2="42.5" y2="42.25" width="0.2" layer="1"/>
 <wire x1="42.5" y1="42.25" x2="40" y2="42.25" width="0.2" layer="1"/>
@@
 <wire x1="36.75" y1="39" x2="36.75" y2="34.510665625" width="0.2" layer="1"/>
 <wire x1="36.75" y1="34.510665625" x2="36.7446" y2="34.2138" width="0.2" layer="1"/>
+<contactref element="U$2" pad="CSN"/>
+<wire x1="43.25" y1="41.5" x2="44.6113" y2="41.5" width="0.2" layer="1"/>
+<wire x1="44.6113" y1="41.5" x2="44.6113" y2="41.5102" width="0.2" layer="1"/>
 </signal>
 <signal name="N$21">
 <contactref element="U2" pad="11"/>
-<contactref element="U$1" pad="5"/>
-<wire x1="44.4" y1="42.75" x2="40" y2="42.75" width="0.2" layer="1"/>
 <wire x1="40" y1="42.75" x2="36.25" y2="39" width="0.2" layer="1"/>
 <wire x1="36.25" y1="39" x2="36.25" y2="34.493265625" width="0.2" layer="1"/>
 <wire x1="36.25" y1="34.493265625" x2="36.262" y2="34.2138" width="0.2" layer="1"/>
+<contactref element="U$2" pad="SCK"/>
+<wire x1="40" y1="42.75" x2="44.6113" y2="42.75" width="0.2" layer="1"/>
+<wire x1="44.6113" y1="42.75" x2="44.6113" y2="42.7802" width="0.2" layer="1"/>
 </signal>
 <signal name="N$37">
 <contactref element="U2" pad="13"/>
-<contactref element="U$1" pad="7"/>
-<wire x1="44.4" y1="45.3" x2="43.3" y2="45.3" width="0.2" layer="1"/>
 <wire x1="43.3" y1="45.3" x2="43" y2="45" width="0.2" layer="1"/>
 <wire x1="43" y1="45" x2="43" y2="44.25" width="0.2" layer="1"/>
@@
 <wire x1="35.25" y1="39" x2="35.25" y2="34.509265625" width="0.2" layer="1"/>
 <wire x1="35.25" y1="34.509265625" x2="35.246" y2="34.2138" width="0.2" layer="1"/>
+<contactref element="U$2" pad="MISO"/>
+<wire x1="43.3" y1="45.3" x2="44.6113" y2="45.3" width="0.2" layer="1"/>
+<wire x1="44.6113" y1="45.3" x2="44.6113" y2="45.3202" width="0.2" layer="1"/>
 </signal>
 <signal name="N$13">
@@
 <contactref element="U2" pad="26"/>
 <wire x1="29.275" y1="17.025" x2="29.275" y2="18.25" width="0.2" layer="1"/>
-<wire x1="29.275" y1="18.25" x2="33.5" y2="18.25" width="0.2" layer="1"/>
-<wire x1="33.5" y1="18.25" x2="34.25" y2="19" width="0.2" layer="1"/>
-<wire x1="34.25" y1="19" x2="34.25" y2="19.5" width="0.2" layer="1"/>
-<wire x1="34.25" y1="19.5" x2="34.2554" y2="20.7446" width="0.2" layer="1"/>
+<wire x1="29.275" y1="18.25" x2="32.5" y2="18.25" width="0.2" layer="1"/>
+<wire x1="32.75" y1="18.25" x2="33.5" y2="18.25" width="0" layer="19" extent="1-16"/>
+<wire x1="34.25" y1="19.75" x2="34.2554" y2="20.7446" width="0.2" layer="1"/>
 <wire x1="34.2554" y1="20.7446" x2="34.2554" y2="29.2862" width="0.2" layer="1"/>
+<wire x1="34.25" y1="19.75" x2="32.5" y2="19.75" width="0.2" layer="1"/>
+<wire x1="32.5" y1="19.75" x2="32.5" y2="18.25" width="0.2" layer="1"/>
+<wire x1="32.5" y1="18.25" x2="32.75" y2="18.25" width="0" layer="19" extent="1-16"/>
 </signal>
 <signal name="N$17">
@@
 <wire x1="29.275" y1="14.975" x2="28.75" y2="15.5" width="0.2" layer="1"/>
 <wire x1="28.75" y1="15.5" x2="28.75" y2="18.75" width="0.2" layer="1"/>
-<wire x1="28.75" y1="18.75" x2="33" y2="18.75" width="0.2" layer="1"/>
-<wire x1="33" y1="18.75" x2="33.75" y2="19.5" width="0.2" layer="1"/>
-<wire x1="33.75" y1="19.5" x2="33.75" y2="29.2836" width="0.2" layer="1"/>
+<wire x1="28.75" y1="18.75" x2="32" y2="18.75" width="0.2" layer="1"/>
+<wire x1="32" y1="18.75" x2="33" y2="18.75" width="0" layer="19" extent="1-16"/>
+<wire x1="33.75" y1="20.25" x2="33.75" y2="29.2836" width="0.2" layer="1"/>
 <wire x1="33.75" y1="29.2836" x2="33.7474" y2="29.2862" width="0.2" layer="1"/>
+<wire x1="33.75" y1="20.25" x2="32" y2="20.25" width="0.2" layer="1"/>
+<wire x1="32" y1="20.25" x2="32" y2="18.75" width="0.2" layer="1"/>
 </signal>
 <signal name="N$23">
@@
 <signal name="N$1">
 <contactref element="U2" pad="12"/>
-<contactref element="U$1" pad="6"/>
-<wire x1="44.4" y1="44.05" x2="43.3" y2="44.05" width="0.2" layer="1"/>
 <wire x1="43.3" y1="44.05" x2="42.5" y2="43.25" width="0.2" layer="1"/>
 <wire x1="42.5" y1="43.25" x2="40" y2="43.25" width="0.2" layer="1"/>
@@
 <wire x1="35.75" y1="39" x2="35.75" y2="34.501265625" width="0.2" layer="1"/>
 <wire x1="35.75" y1="34.501265625" x2="35.754" y2="34.2138" width="0.2" layer="1"/>
+<contactref element="U$2" pad="MOSI"/>
+<wire x1="43.3" y1="44.05" x2="44.6113" y2="44.05" width="0.2" layer="1"/>
+<wire x1="44.6113" y1="44.05" x2="44.6113" y2="44.0502" width="0.2" layer="1"/>
 </signal>
 <signal name="N$2">
