File: client/eagle_proj/jake_client.sch (EAGLE design)
At the start: 12 parts, among them IC1 BME280, U2 ATMEGA328P-MU, U3 APDS-9960, U4 RPI-103X

Commit message: Clared client todo
Parts:
- removed U$1: NRF24L01+, NRF:NRF24L01+
- added R1: 10k, SparkFun:RESISTOR0402-RES
- added U$2: NRF24L01+NRF24L01+MINI, nrf24L01:NRF24L01+NRF24L01+MINI
Connections:
- net N$1: now also U$2.MOSI; no longer U$1.6.MOSI
- net N$14: now also R1.1
- net N$18: now also U$2.CE; no longer U$1.3.CE
- net N$19: now also U$2.CSN; no longer U$1.4.CSN
- net N$21: now also U$2.SCK; no longer U$1.5.SCK
- net N$37: now also U$2.MISO; no longer U$1.7.MISO
- net VCC: now also R1.2
Changed lines of the file:
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@@
 <part name="GND16" library="SparkFun" deviceset="GND" device=""/>
 <part name="R3" library="SparkFun" deviceset="RESISTOR" device="0402-RES" value="39"/>
-<part name="U$1" library="NRF" deviceset="NRF24L01+" device=""/>
 <part name="V1" library="battery_xtra" deviceset="TAKACHI_BATT" device="-CR123A"/>
+<part name="U$2" library="nrf24L01" deviceset="NRF24L01+" device="NRF24L01+MINI"/>
+<part name="R1" library="SparkFun" deviceset="RESISTOR" device="0402-RES" value="10k"/>
 </parts>
 <sheets>
@@
 <instance part="GND16" gate="1" x="157.48" y="165.1"/>
 <instance part="R3" gate="G$1" x="142.24" y="167.64"/>
-<instance part="U$1" gate="G$1" x="137.16" y="96.52"/>
 <instance part="V1" gate="G$1" x="0" y="154.94" smashed="yes" rot="R90">
 <attribute name="NAME" x="-3.175" y="153.67" size="1.778" layer="95" rot="R90"/>
 <attribute name="VALUE" x="4.445" y="153.67" size="1.27" layer="96" rot="R90"/>
 </instance>
+<instance part="U$2" gate="G$1" x="154.94" y="104.14"/>
+<instance part="R1" gate="G$1" x="101.6" y="66.04"/>
 </instances>
 <busses>
@@
 <pinref part="P1" gate="A" pin="2"/>
 <wire x1="101.6" y1="55.88" x2="111.76" y2="55.88" width="0.1524" layer="91"/>
+<wire x1="111.76" y1="58.42" x2="109.22" y2="58.42" width="0.1524" layer="91"/>
+<wire x1="109.22" y1="58.42" x2="109.22" y2="66.04" width="0.1524" layer="91"/>
+<junction x="111.76" y="58.42"/>
+<pinref part="R1" gate="G$1" pin="2"/>
+<wire x1="106.68" y1="66.04" x2="109.22" y2="66.04" width="0.1524" layer="91"/>
 </segment>
 <segment>
@@
 <pinref part="U2" gate="A" pin="PB3"/>
 <wire x1="91.44" y1="93.98" x2="71.12" y2="93.98" width="0.1524" layer="91"/>
-<wire x1="83.82" y1="60.96" x2="83.82" y2="68.58" width="0.1524" layer="91"/>
-<wire x1="83.82" y1="68.58" x2="91.44" y2="68.58" width="0.1524" layer="91"/>
-<wire x1="91.44" y1="68.58" x2="91.44" y2="93.98" width="0.1524" layer="91"/>
-<wire x1="114.3" y1="63.5" x2="109.22" y2="63.5" width="0.1524" layer="91"/>
-<wire x1="114.3" y1="53.34" x2="114.3" y2="63.5" width="0.1524" layer="91"/>
-<wire x1="83.82" y1="60.96" x2="109.22" y2="60.96" width="0.1524" layer="91"/>
-<wire x1="109.22" y1="60.96" x2="109.22" y2="63.5" width="0.1524" layer="91"/>
+<wire x1="91.44" y1="71.12" x2="91.44" y2="93.98" width="0.1524" layer="91"/>
+<wire x1="114.3" y1="53.34" x2="114.3" y2="71.12" width="0.1524" layer="91"/>
+<wire x1="91.44" y1="71.12" x2="114.3" y2="71.12" width="0.1524" layer="91"/>
 <pinref part="P1" gate="A" pin="4"/>
 <wire x1="101.6" y1="53.34" x2="114.3" y2="53.34" width="0.1524" layer="91"/>
@@
 <net name="N$14" class="0">
 <segment>
-<wire x1="58.42" y1="50.8" x2="58.42" y2="83.82" width="0.1524" layer="91"/>
+<wire x1="58.42" y1="50.8" x2="58.42" y2="66.04" width="0.1524" layer="91"/>
 <pinref part="P1" gate="A" pin="5"/>
+<wire x1="58.42" y1="66.04" x2="58.42" y2="83.82" width="0.1524" layer="91"/>
 <wire x1="93.98" y1="50.8" x2="58.42" y2="50.8" width="0.1524" layer="91"/>
 <pinref part="U2" gate="A" pin="PC6"/>
 <wire x1="35.56" y1="86.36" x2="35.56" y2="83.82" width="0.1524" layer="91"/>
 <wire x1="35.56" y1="83.82" x2="58.42" y2="83.82" width="0.1524" layer="91"/>
+<pinref part="R1" gate="G$1" pin="1"/>
+<wire x1="58.42" y1="66.04" x2="96.52" y2="66.04" width="0.1524" layer="91"/>
+<junction x="58.42" y="66.04"/>
 </segment>
 </net>
@@
 <wire x1="71.12" y1="111.76" x2="111.76" y2="111.76" width="0.1524" layer="91"/>
 <wire x1="111.76" y1="111.76" x2="111.76" y2="106.68" width="0.1524" layer="91"/>
-<pinref part="U$1" gate="G$1" pin="3.CE"/>
-<wire x1="111.76" y1="106.68" x2="114.3" y2="106.68" width="0.1524" layer="91"/>
+<wire x1="142.24" y1="100.33" x2="127" y2="100.33" width="0.1524" layer="91"/>
+<wire x1="127" y1="100.33" x2="127" y2="106.68" width="0.1524" layer="91"/>
+<wire x1="127" y1="106.68" x2="111.76" y2="106.68" width="0.1524" layer="91"/>
+<pinref part="U$2" gate="G$1" pin="CE"/>
 </segment>
 </net>
@@
 <wire x1="109.22" y1="109.22" x2="71.12" y2="109.22" width="0.1524" layer="91"/>
 <wire x1="109.22" y1="109.22" x2="109.22" y2="101.6" width="0.1524" layer="91"/>
-<pinref part="U$1" gate="G$1" pin="4.CSN"/>
-<wire x1="109.22" y1="101.6" x2="114.3" y2="101.6" width="0.1524" layer="91"/>
+<wire x1="142.24" y1="97.79" x2="124.46" y2="97.79" width="0.1524" layer="91"/>
+<wire x1="124.46" y1="97.79" x2="124.46" y2="101.6" width="0.1524" layer="91"/>
+<wire x1="124.46" y1="101.6" x2="109.22" y2="101.6" width="0.1524" layer="91"/>
+<pinref part="U$2" gate="G$1" pin="CSN"/>
 </segment>
 </net>
@@
 <wire x1="106.68" y1="106.68" x2="71.12" y2="106.68" width="0.1524" layer="91"/>
 <wire x1="106.68" y1="106.68" x2="106.68" y2="96.52" width="0.1524" layer="91"/>
-<pinref part="U$1" gate="G$1" pin="5.SCK"/>
-<wire x1="106.68" y1="96.52" x2="114.3" y2="96.52" width="0.1524" layer="91"/>
+<wire x1="106.68" y1="96.52" x2="116.84" y2="96.52" width="0.1524" layer="91"/>
+<wire x1="170.18" y1="105.41" x2="177.8" y2="105.41" width="0.1524" layer="91"/>
+<wire x1="177.8" y1="105.41" x2="177.8" y2="91.44" width="0.1524" layer="91"/>
+<wire x1="177.8" y1="91.44" x2="124.46" y2="91.44" width="0.1524" layer="91"/>
+<wire x1="124.46" y1="91.44" x2="124.46" y2="93.98" width="0.1524" layer="91"/>
+<wire x1="124.46" y1="93.98" x2="116.84" y2="93.98" width="0.1524" layer="91"/>
+<wire x1="116.84" y1="93.98" x2="116.84" y2="96.52" width="0.1524" layer="91"/>
+<pinref part="U$2" gate="G$1" pin="SCK"/>
 </segment>
 </net>
@@
 <wire x1="101.6" y1="99.06" x2="71.12" y2="99.06" width="0.1524" layer="91"/>
 <wire x1="101.6" y1="99.06" x2="101.6" y2="86.36" width="0.1524" layer="91"/>
-<pinref part="U$1" gate="G$1" pin="7.MISO"/>
-<wire x1="101.6" y1="86.36" x2="114.3" y2="86.36" width="0.1524" layer="91"/>
+<wire x1="101.6" y1="86.36" x2="116.84" y2="86.36" width="0.1524" layer="91"/>
+<wire x1="170.18" y1="100.33" x2="172.72" y2="100.33" width="0.1524" layer="91"/>
+<wire x1="172.72" y1="100.33" x2="172.72" y2="83.82" width="0.1524" layer="91"/>
+<wire x1="172.72" y1="83.82" x2="116.84" y2="83.82" width="0.1524" layer="91"/>
+<wire x1="116.84" y1="83.82" x2="116.84" y2="86.36" width="0.1524" layer="91"/>
+<pinref part="U$2" gate="G$1" pin="MISO"/>
 </segment>
 </net>
@@
 <wire x1="71.12" y1="101.6" x2="104.14" y2="101.6" width="0.1524" layer="91"/>
 <wire x1="104.14" y1="101.6" x2="104.14" y2="91.44" width="0.1524" layer="91"/>
-<pinref part="U$1" gate="G$1" pin="6.MOSI"/>
-<wire x1="104.14" y1="91.44" x2="114.3" y2="91.44" width="0.1524" layer="91"/>
-</segment>
-</net>
+<wire x1="104.14" y1="91.44" x2="116.84" y2="91.44" width="0.1524" layer="91"/>
+<wire x1="170.18" y1="102.87" x2="175.26" y2="102.87" width="0.1524" layer="91"/>
+<wire x1="175.26" y1="102.87" x2="175.26" y2="88.9" width="0.1524" layer="91"/>
+<wire x1="175.26" y1="88.9" x2="116.84" y2="88.9" width="0.1524" layer="91"/>
+<wire x1="116.84" y1="88.9" x2="116.84" y2="91.44" width="0.1524" layer="91"/>
+<pinref part="U$2" gate="G$1" pin="MOSI"/>
+</segment>
+</net>
